Commit message: training DQN states

File: UWRTArmGym/urdf/arm.urdf.xacro (robot description, xacro)
@@ -228,5 +228,5 @@
       <origin xyz="0 0 ${forearm_length + 0.01}"
               rpy="0 0 0"/>
-      <axis xyz="0 0 1"/>
+      <axis xyz="1 0 0"/>
       <limit lower="${wrist_roll_min_angle * M_PI / 180.0}"
              upper="${wrist_roll_max_angle * M_PI / 180.0}"

File: UWRTArmGym/urdf/uwrt_arm.urdf (robot description, URDF)
Before this commit: robot uwrt_arm, 7 links, 6 joints
Joints:
- joint arm_wrist_roll_joint: axis 0 0 1 -> 1 0 0
